File: hardware/AtomLinkMini-PCB/AtomLinkMini-PCB.kicad_sch (KiCad schematic)
At the start: 23 parts, among them J1 PF cable, J2 Servo, J3 Grove cable, Q1 AS2309, Q2 MUN5235, Q3 AS2309, Q4 MUN5235, SW1 SW_SPST, U1 ATtiny13A-SS

Commit message: Added atTiny13 schematic PDF, rewired schematic for atTiny402 & generated PDF
Parts:
- removed U1: ATtiny13A-SS, Package_SO:SOIC-8_3.9x4.9mm_P1.27mm, symbol MCU_Microchip_ATtiny:ATtiny13A-SS
- added U?: (no value), symbol MCU_Microchip_ATtiny:ATtiny402-SS
- C2: value (none) -> 10u; footprint (none) -> Capacitor_SMD:C_0805_2012Metric_Pad1.18x1.45mm_HandSolder
- TP1: value debugWire -> (none)
Connections:
- net +5V: now also U?.1 (VCC)
- net Button: now also U?.3 (PA7)
- net GND: now also U?.8 (GND)
- net LED: now also U?.4 (PA1)
- net PF_M1_TTL: now also U?.5 (PA2)
- net PF_M2_TTL: now also U?.2 (PA6)
- net Servo: now also U?.7 (PA3)
- net dW renamed UPDI
- net UPDI: now also U?.6 (~{RESET}/PA0)
Other:
- moved on the sheet: R1, TP1
